Commit message: fix(ekf, rviz, lidar): eliminate odometry drift by removing ax integration, fix lidar height and point size

File: tank_description/urdf/lidar.xacro (robot description, xacro)
@@ -1,9 +1,9 @@
 <?xml version="1.0"?>
 <robot xmlns:xacro="http://www.ros.org/wiki/xacro">
-  <!-- RPLIDAR A2M12 Mount on Top of Chassis -->
+  <!-- RPLIDAR A2M12 Mount on Top of Chassis (Clearance above chassis to prevent self-collision) -->
   <joint name="laser_joint" type="fixed">
     <parent link="base_link"/>
     <child link="laser_frame"/>
-    <origin xyz="0.06 0.0 0.09" rpy="0 0 0"/>
+    <origin xyz="0.06 0.0 0.11" rpy="0 0 0"/>
   </joint>
   <link name="laser_frame">
